Commit message: added parse and publish

File: urdf/braccio_arm.urdf (robot description, URDF)
Before this commit: robot braccio, 8 links, 7 joints
Joints:
- joint base_joint: axis 0 0 -1 -> 0 0 1
- joint gripper_joint: limit lower=1.217 upper=1.5708 effort=1000.0 velocity=1.0 -> lower=0.1750 upper=1.2741 effort=1000.0 velocity=1.0; origin xyz=0.010 0 0.03 rpy=0 0 0 -> xyz=0.010 0 0.03 rpy=0 -0.2967 0
- joint sub_gripper_joint: limit lower=1.5708 upper=2.7876 effort=1000.0 velocity=1.0 -> lower=1.2741 upper=2.3732 effort=1000.0 velocity=1.0; origin xyz=-0.010 0 0.03 rpy=0 3.1416 0 -> xyz=-0.010 0 0.03 rpy=0 3.4383 0
- joint wrist_roll_joint: origin xyz=0 0.0 0.06 rpy=0 0 0 -> xyz=0 0.0 0.06 rpy=0 0 1.5708

Commit message: changed name

File: urdf/braccio_arm.urdf (robot description, URDF)
Before this commit: robot braccio, 8 links, 7 joints
Links:
- link braccio_base_link: geometry visual mesh filename=package://braccio_arduino_ros_rviz/stl/braccio_base.stl scale=0.001 0.001 0.001
- link elbow_link: geometry visual mesh filename=package://braccio_arduino_ros_rviz/stl/braccio_elbow.stl scale=0.001 0.001 0.001
- link left_gripper_link: geometry visual mesh filename=package://braccio_arduino_ros_rviz/stl/braccio_left_gripper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 scale=0.001 0.001 0.001
- link right_gripper_link: geometry visual mesh filename=package://braccio_arduino_ros_rviz/stl/braccio_right_grippe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 scale=0.001 0.001 0.001
- link shoulder_link: geometry visual mesh filename=package://braccio_arduino_ros_rviz/stl/braccio_shoulder.stl scale=0.001 0.001 0.001
- link wrist_pitch_link: geometry visual mesh filename=package://braccio_arduino_ros_rviz/stl/braccio_wrist_pitch.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 scale=0.001 0.001 0.001
- link wrist_roll_link: geometry visual mesh filename=package://braccio_arduino_ros_rviz/stl/braccio_wrist_roll.s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 scale=0.001 0.001 0.001
